File: Engineering 2023 UAV flight controller/Engineering 2023 UAV flight controller.kicad_sch (KiCad schematic)
At the start: 12 parts

Commit message: dont remember changes, were last night
Parts:
- removed J?: Aileron Right, symbol Connector_Generic:Conn_01x03
- removed J?: Elevator Left, symbol Connector_Generic:Conn_01x03
- removed J?: Elevator Right, symbol Connector_Generic:Conn_01x03
- removed J?: Aileron Left, symbol Connector_Generic:Conn_01x03
- removed U?: MPU-6500, QFN24_3X3X0P9_IVS, symbol MPU-6500:MPU-6500
- removed U?: SX1280IMLTRT, QFN24_4X4_SEM, symbol SX1280:SX1280IMLTRT
- added M?: elevator Left, symbol Motor:Motor_Servo
- added M?: elevator Right, symbol Motor:Motor_Servo
- added M?: aileron Right, symbol Motor:Motor_Servo
- added M?: aileron Left, symbol Motor:Motor_Servo
- added U?: MMC5983MA, MMC5983MA_MEM, symbol MMC5983MA:MMC5983MA
- added U?: MPU-6050, Sensor_Motion:InvenSense_QFN-24_4x4mm_P0.5mm, symbol Sensor_Motion:MPU-6050
- J?: footprint (none) -> Connector_USB:USB_C_Receptacle_JAE_DX07S016JA1R1500

Commit message: some small updates
Parts:
- M?: value elevator Left -> Elevator Left
- M?: value elevator Right -> Elevator Right
- M?: value aileron Right -> Aileron Right
- M?: value aileron Left -> Aileron Left
Connections:
- net Elevator Left PWM: now reaches M?.1 (PWM)
- net Elevator Right PWM: now reaches M?.1 (PWM)
- net Aileron Right PWM: now reaches M?.1 (PWM)
- net Aileron Left PWM: now reaches M?.1 (PWM)
- net ESC PWM: now reaches J?.1 (Pin_1)
- net ESC positive rail: now reaches J?.2 (Pin_2)
- net ESC negitive rail: now reaches J?.3 (Pin_3)
Other:
- moved on the sheet: J?, U?
Changed lines of the file:
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@@
 (kicad_sch (version 20211123) (generator eeschema)
   (paper "A3")
+  (wire (pts (xy 368.3 50.8) (xy 388.62 50.8))
+    (stroke (width 0) (type default) (color 0 0 0 0))
+  )
+  (wire (pts (xy 368.3 63.5) (xy 388.62 63.5))
+    (stroke (width 0) (type default) (color 0 0 0 0))
+  )
+  (wire (pts (xy 368.3 26.67) (xy 388.62 26.67))
+    (stroke (width 0) (type default) (color 0 0 0 0))
+  )
+  (wire (pts (xy 368.3 38.1) (xy 388.62 38.1))
+    (stroke (width 0) (type default) (color 0 0 0 0))
+  )
+  (wire (pts (xy 368.3 66.04) (xy 388.62 66.04))
+    (stroke (width 0) (type default) (color 0 0 0 0))
+  )
+  (wire (pts (xy 368.3 15.24) (xy 388.62 15.24))
+    (stroke (width 0) (type default) (color 0 0 0 0))
+  )
+  (wire (pts (xy 368.3 68.58) (xy 388.62 68.58))
+    (stroke (width 0) (type default) (color 0 0 0 0))
+  )
+  (label "Elevator Right PWM" (at 368.3 50.8 0)
+    (effects (font (size 1.27 1.27)) (justify left bottom))
+  )
+  (label "Aileron Left PWM" (at 368.3 15.24 0)
+    (effects (font (size 1.27 1.27)) (justify left bottom))
+  )
+  (label "ESC positive rail" (at 368.3 66.04 0)
+    (effects (font (size 1.27 1.27)) (justify left bottom))
+  )
+  (label "Elevator Left PWM" (at 368.3 38.1 0)
+    (effects (font (size 1.27 1.27)) (justify left bottom))
+  )
+  (label "ESC PWM" (at 368.3 63.5 0)
+    (effects (font (size 1.27 1.27)) (justify left bottom))
+  )
+  (label "ESC negitive rail" (at 368.3 68.58 0)
+    (effects (font (size 1.27 1.27)) (justify left bottom))
+  )
+  (label "Aileron Right PWM" (at 368.3 26.67 0)
+    (effects (font (size 1.27 1.27)) (justify left bottom))
+  )
   (symbol (lib_id "Motor:Motor_Servo") (at 396.24 40.64 0) (unit 1)
     (in_bom yes) (on_board yes)
@@
       (effects (font (size 1.27 1.27)) (justify left))
     )
-    (property "Value" "elevator Left" (id 1) (at 391.16 45.72 0)
+    (property "Value" "Elevator Left" (id 1) (at 388.62 45.72 0)
       (effects (font (size 1.27 1.27)) (justify left))
     )
@@
       (effects (font (size 1.27 1.27)) (justify left))
     )
-    (property "Value" "elevator Right" (id 1) (at 391.16 58.42 0)
+    (property "Value" "Elevator Right" (id 1) (at 388.62 58.42 0)
       (effects (font (size 1.27 1.27)) (justify left))
     )
@@
     (pin "S1")
   )
-  (symbol (lib_id "Sensor_Motion:MPU-6050") (at 220.98 87.63 0) (unit 1)
-    (in_bom yes) (on_board yes) (fields_autoplaced)
-    (property "Reference" "U?" (id 0) (at 222.9994 104.14 0)
-      (effects (font (size 1.27 1.27)) (justify left))
-    )
-    (property "Value" "MPU-6050" (id 1) (at 222.9994 106.68 0)
-      (effects (font (size 1.27 1.27)) (justify left))
-    )
-    (property "Footprint" "Sensor_Motion:InvenSense_QFN-24_4x4mm_P0.5mm" (id 2) (at 220.98 107.95 0)
-      (effects (font (size 1.27 1.27)) hide)
-    )
-    (property "Datasheet" "https://store.invensense.com/datasheets/invensense/MPU-6050_DataSheet_V3%204.pdf" (id 3) (at 220.98 91.44 0)
+  (symbol (lib_id "Sensor_Motion:MPU-6050") (at 229.87 88.9 0) (unit 1)
+    (in_bom yes) (on_board yes) (fields_autoplaced)
+    (property "Reference" "U?" (id 0) (at 231.8894 105.41 0)
+      (effects (font (size 1.27 1.27)) (justify left))
+    )
+    (property "Value" "MPU-6050" (id 1) (at 231.8894 107.95 0)
+      (effects (font (size 1.27 1.27)) (justify left))
+    )
+    (property "Footprint" "Sensor_Motion:InvenSense_QFN-24_4x4mm_P0.5mm" (id 2) (at 229.87 109.22 0)
+      (effects (font (size 1.27 1.27)) hide)
+    )
+    (property "Datasheet" "https://store.invensense.com/datasheets/invensense/MPU-6050_DataSheet_V3%204.pdf" (id 3) (at 229.87 92.71 0)
       (effects (font (size 1.27 1.27)) hide)
     )
@@
       (effects (font (size 1.27 1.27)) (justify left))
     )
-    (property "Value" "aileron Right" (id 1) (at 391.16 34.29 0)
+    (property "Value" "Aileron Right" (id 1) (at 388.62 34.29 0)
       (effects (font (size 1.27 1.27)) (justify left))
     )
@@
     (pin "3")
   )
-  (symbol (lib_id "Connector:Micro_SD_Card") (at 34.29 104.14 0) (mirror y) (unit 1)
-    (in_bom yes) (on_board yes) (fields_autoplaced)
-    (property "Reference" "J?" (id 0) (at 33.655 85.09 0))
-    (property "Value" "Micro_SD_Card" (id 1) (at 33.655 87.63 0))
-    (property "Footprint" "" (id 2) (at 5.08 96.52 0)
-      (effects (font (size 1.27 1.27)) hide)
-    )
-    (property "Datasheet" "http://katalog.we-online.de/em/datasheet/693072010801.pdf" (id 3) (at 34.29 104.14 0)
+  (symbol (lib_id "Connector:Micro_SD_Card") (at 247.65 144.78 0) (mirror x) (unit 1)
+    (in_bom yes) (on_board yes) (fields_autoplaced)
+    (property "Reference" "J?" (id 0) (at 248.285 123.19 0))
+    (property "Value" "Micro_SD_Card" (id 1) (at 248.285 125.73 0))
+    (property "Footprint" "" (id 2) (at 276.86 152.4 0)
+      (effects (font (size 1.27 1.27)) hide)
+    )
+    (property "Datasheet" "http://katalog.we-online.de/em/datasheet/693072010801.pdf" (id 3) (at 247.65 144.78 0)
       (effects (font (size 1.27 1.27)) hide)
     )
@@
       (effects (font (size 1.27 1.27)) (justify left))
     )
-    (property "Value" "aileron Left" (id 1) (at 391.16 22.86 0)
+    (property "Value" "Aileron Left" (id 1) (at 388.62 22.86 0)
       (effects (font (size 1.27 1.27)) (justify left))
     )
@@
     (pin "3")
   )
-  (symbol (lib_id "RF_GPS:NEO-M8N") (at 317.5 157.48 0) (unit 1)
-    (in_bom yes) (on_board yes) (fields_autoplaced)
-    (property "Reference" "U?" (id 0) (at 319.5194 180.34 0)
-      (effects (font (size 1.27 1.27)) (justify left))
-    )
-    (property "Value" "NEO-M8N" (id 1) (at 319.5194 182.88 0)
-      (effects (font (size 1.27 1.27)) (justify left))
-    )
-    (property "Footprint" "RF_GPS:ublox_NEO" (id 2) (at 327.66 179.07 0)
-      (effects (font (size 1.27 1.27)) hide)
-    )
-    (property "Datasheet" "https://www.u-blox.com/sites/default/files/NEO-M8-FW3_DataSheet_%28UBX-15031086%29.pdf" (id 3) (at 317.5 157.48 0)
+  (symbol (lib_id "RF_GPS:NEO-M8N") (at 365.76 205.74 0) (unit 1)
+    (in_bom yes) (on_board yes) (fields_autoplaced)
+    (property "Reference" "U?" (id 0) (at 367.7794 228.6 0)
+      (effects (font (size 1.27 1.27)) (justify left))
+    )
+    (property "Value" "NEO-M8N" (id 1) (at 367.7794 231.14 0)
+      (effects (font (size 1.27 1.27)) (justify left))
+    )
+    (property "Footprint" "RF_GPS:ublox_NEO" (id 2) (at 375.92 227.33 0)
+      (effects (font (size 1.27 1.27)) hide)
+    )
+    (property "Datasheet" "https://www.u-blox.com/sites/default/files/NEO-M8-FW3_DataSheet_%28UBX-15031086%29.pdf" (id 3) (at 365.76 205.74 0)
       (effects (font (size 1.27 1.27)) hide)
     )
@@
     (pin "9")
   )
-  (symbol (lib_id "Connector_Generic:Conn_01x03") (at 393.7 68.58 0) (unit 1)
+  (symbol (lib_id "Connector_Generic:Conn_01x03") (at 393.7 66.04 0) (unit 1)
     (in_bom yes) (on_board yes)
-    (property "Reference" "J?" (id 0) (at 396.24 67.3099 0)
-      (effects (font (size 1.27 1.27)) (justify left))
-    )
-    (property "Value" "ESC speed control" (id 1) (at 388.62 74.93 0)
-      (effects (font (size 1.27 1.27)) (justify left))
-    )
-    (property "Footprint" "" (id 2) (at 393.7 68.58 0)
-      (effects (font (size 1.27 1.27)) hide)
-    )
-    (property "Datasheet" "~" (id 3) (at 393.7 68.58 0)
+    (property "Reference" "J?" (id 0) (at 396.24 64.7699 0)
+      (effects (font (size 1.27 1.27)) (justify left))
+    )
+    (property "Value" "ESC speed control" (id 1) (at 388.62 72.39 0)
+      (effects (font (size 1.27 1.27)) (justify left))
+    )
+    (property "Footprint" "" (id 2) (at 393.7 66.04 0)
+      (effects (font (size 1.27 1.27)) hide)
+    )
+    (property "Datasheet" "~" (id 3) (at 393.7 66.04 0)
       (effects (font (size 1.27 1.27)) hide)
     )
@@
     )
     (path "/10ec48c8-c7b5-43a4-bb63-38ddcdfa745e"
-      (reference "M?") (unit 1) (value "elevator Left") (footprint "")
+      (reference "M?") (unit 1) (value "Elevator Left") (footprint "")
     )
     (path "/4e2503e3-7522-4959-b540-6c7684261f30"
-      (reference "M?") (unit 1) (value "elevator Right") (footprint "")
+      (reference "M?") (unit 1) (value "Elevator Right") (footprint "")
     )
     (path "/a5803e7c-8b9f-45cb-9ce9-ade452865f1b"
-      (reference "M?") (unit 1) (value "aileron Right") (footprint "")
+      (reference "M?") (unit 1) (value "Aileron Right") (footprint "")
     )
     (path "/d40a1cc5-fbc2-4c1e-9349-e721bb07408e"
-      (reference "M?") (unit 1) (value "aileron Left") (footprint "")
+      (reference "M?") (unit 1) (value "Aileron Left") (footprint "")
     )
     (path "/357beecd-919b-401e-b840-f3b5be37c3a3"

Commit message: added a symbol for the (symbol "E28-2G4M27S" (in_bom yes) (on_board yes)   (property "Reference" "U" (id 0) (at 0 0 0)     (effects (font (size 1.27 1.27)))   )   (property "Value" "E28-2G4M27S" (id 1) (at 6.35 2.54 0)     (effects (font (size 1.27 1.27)))   )   (property "Footprint" "" (id 2) (at 0 0 0)     (effects (font (size 1.27 1.27)) hide)   )   (property "Datasheet" "" (id 3) (at 0 0 0)     (effects (font (size 1.27 1.27)) hide)   )   (symbol "E28-2G4M27S_1_1"     (pin input line (at 2.54 -5.08 0) (length 2.54)       (name "GND" (effects (font (size 1.27 1.27))))       (number "" (effects (font (size 1.27 1.27))))     )   ) ) ... yeh that
Parts:
- added U?: E28-2G4M27S, symbol SX1280:E28-2G4M27S
Changed lines of the file:
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@@
     (pin "3")
+  )
+  (symbol (lib_id "SX1280:E28-2G4M27S") (at 236.22 163.83 0) (unit 1)
+    (in_bom yes) (on_board yes) (fields_autoplaced)
+    (property "Reference" "U?" (id 0) (at 275.0694 181.61 0)
+      (effects (font (size 1.27 1.27)) (justify left))
+    )
+    (property "Value" "E28-2G4M27S" (id 1) (at 275.0694 184.15 0)
+      (effects (font (size 1.27 1.27)) (justify left))
+    )
+    (property "Footprint" "" (id 2) (at 236.22 163.83 0)
+      (effects (font (size 1.27 1.27)) hide)
+    )
+    (property "Datasheet" "" (id 3) (at 236.22 163.83 0)
+      (effects (font (size 1.27 1.27)) hide)
+    )
+    (pin "1")
+    (pin "10")
+    (pin "11")
+    (pin "12")
+    (pin "13")
+    (pin "14")
+    (pin "15")
+    (pin "16")
+    (pin "2")
+    (pin "3")
+    (pin "4")
+    (pin "5")
+    (pin "6")
+    (pin "7")
+    (pin "8")
+    (pin "9")
   )
   (symbol (lib_id "MMC5983MA:MMC5983MA") (at 251.46 64.77 0) (unit 1)
@@
       (reference "M?") (unit 1) (value "Aileron Left") (footprint "")
     )
+    (path "/2fad4847-f932-40e7-a067-d76f37f4cf43"
+      (reference "U?") (unit 1) (value "E28-2G4M27S") (footprint "")
+    )
     (path "/357beecd-919b-401e-b840-f3b5be37c3a3"

Commit message: E
Parts:
- added U?: LPS25HB, Package_LGA:ST_HLGA-10_2.5x2.5mm_P0.6mm_LayoutBorder3x2y, symbol Sensor_Pressure:LPS25HB
Connections:
- net ESC negitive rail is gone; now on net GND: J?.3 (Pin_3)
- net Servo 6V rail: now reaches M?.2 (+)
- net Servo 6V rail: now also M?.2 (+), M?.2 (+), M?.2 (+)
- net GND: now reaches M?.3 (-)
- net GND: now also M?.3 (-), M?.3 (-), M?.3 (-)
- new net: U?.3 (GND), U?.8 (GND), U?.9 (GND)
Other:
- note added: "128MB flash"
- note added: "Barometer"
- note added: "External connections"
- note added: "GPS"
- note added: "LORA 2.4GHz"
- note added: "MicroSD card"
- note added: "Periferals"
- note added: "Power"
- note added: "RF connections"
- note added: "RP2040"
- note added: "accel/gyro"
- note added: "mag sensor (compass)"
- moved on the sheet: J?, M?, U?

Commit message: did a little trolling, started on the power supply
Parts:
- added R? (x2): 5k1, symbol Device:R
- added SW?: SW_SPDT, symbol Switch:SW_SPDT
Connections:
- net ESC positive rail: now also SW?.3 (C)
- net GND: now also J?.A1 (GND), J?.A12 (GND), J?.B1 (GND), J?.B12 (GND), J?.S1 (SHIELD), R?.1, R?.1
- net USB_C positive rail: now reaches J?.A4 (VBUS), J?.A9 (VBUS), J?.B4 (VBUS), J?.B9 (VBUS)
- net USB_C positive rail: now also SW?.1 (A)
- net at J?.A5 (CC1): now also R?.2
- net usb+: now reaches J?.A6 (D+)
- net usb+: now also J?.B6 (D+)
- net usb-: now reaches J?.A7 (D-)
- net usb-: now also J?.B7 (D-)
- net at J?.B5 (CC2): now also R?.2
- no-connect marks 0 -> 2
Other:
- note added: "config"
- note added: "dont know what these do"
- note added: "has two of each?"
- moved on the sheet: J?

Commit message: finished power and rp2040 pinout
Parts:
- added C1, C2, C4, C6: 0.1uf, symbol Device:C
- added C10, C11, C13, C15, C16, C17, C18, C19, C20, C7: 100n, symbol Device:C
- added C12, C14: 1u, symbol Device:C
- added C3, C5: 1uf, symbol Device:C
- added C8, C9: 27p, symbol Device:C
- added D1, D2: LED_GREEN, symbol Device:LED
- added D3: LED_RED, symbol Device:LED
- added R1: R, symbol Device:R
- added R10, R11, R6, R7: 330, symbol Device:R
- added R2: R_Trim, symbol Device:R_Trim
- added R5: 1k, symbol Device:R
- added R8, R9: 27.4, symbol Device:R
- added SW2: SW_Push_LED, symbol Switch:SW_Push_LED
- added U2: AMS1117-3.3, Package_TO_SOT_SMD:SOT-223-3_TabPin2, symbol Regulator_Linear:AMS1117-3.3
- added U3: LM350_TO220, Package_TO_SOT_THT:TO-220-3_Vertical, symbol Regulator_Linear:LM350_TO220
- added Y1: ABLS-12.000MHZ-B4-T, symbol Device:Crystal
- gave numbers to parts that had none: 17
Connections:
- net GND: now also U1.4 (GND), U4.19 (TESTEN), U4.57 (GND), C1.2, C10.2, C11.2, C12.2, C13.2, C14.2, C15.2, C16.2, C17.2, C18.2, C19.2, C2.2, C20.2, C3.2, C4.2, C5.2, C6.2, C7.2, C8.1, C9.1, R10.2, R11.2, R2.2, R6.2, R7.2, SW2.1, U2.1 (GND)
- net Servo 6V rail: now also C5.1, C6.1, D3.2 (A), R1.1, U3.2 (VO)
- net USB_C positive rail: now also D1.2 (A)
- net reg in: now reaches SW1.2 (B)
- net reg in: now also C1.1, C2.1, U2.3 (VI), U3.3 (VI)
- net QSPI_SS: now reaches U1.1 (~{CS})
- net QSPI_SS: now also U1.6 (CLK), U4.56 (QSPI_SS), R5.1
- net QSPI_SD1: now reaches U1.2 (DO(IO1))
- net QSPI_SD1: now also U4.55 (QSPI_SD1)
- net QSPI_SD2: now reaches U1.3 (IO2)
- net QSPI_SD2: now also U4.54 (QSPI_SD2)
- net QSPI_SD0: now reaches U1.5 (DI(IO0))
- net QSPI_SD0: now also U4.53 (QSPI_SD0)
- net QSPI_SD3: now reaches U1.7 (IO3)
- net QSPI_SD3: now also U4.51 (QSPI_SD3)
- net 3.3v rail: now reaches U1.8 (VCC)
- net 3.3v rail: now also U4.1 (IOVDD), U4.10 (IOVDD), U4.22 (IOVDD), U4.33 (IOVDD), U4.42 (IOVDD), U4.43 (ADC_AVDD), U4.44 (VREG_IN), U4.48 (USB_VDD), U4.49 (IOVDD), C13.1, C14.1, C15.1, C16.1, C17.1, C18.1, C19.1, C20.1, C3.1, C4.1, C7.1, D2.2 (A), SW2.4 (A), U2.2 (VO)
- net XIN: now reaches U4.20 (XIN)
- net XIN: now also C8.2, Y1.1
- net XOUT: now reaches U4.21 (XOUT)
- net XOUT: now also C9.2, Y1.2
- net 1.1V internal rp2040 reg: now reaches U4.23 (DVDD), U4.50 (DVDD)
- net 1.1V internal rp2040 reg: now also U4.45 (VREG_VOUT), C10.1, C11.1, C12.1
- net SWCLK: now reaches U4.24 (SWCLK)
- net SWD: now reaches U4.25 (SWD)
- net RUN: now reaches U4.26 (RUN)
- net -: now reaches U4.46 (USB_DM)
- net -: now also R9.2
- net +: now reaches U4.47 (USB_DP)
- net +: now also R8.2
- net QSPI_SCLK: now reaches U4.52 (QSPI_SCLK)
- net usb+ renamed USB_DP
- net USB_DP: now also R8.1
- net usb- renamed USB_DM
- net USB_DM: now also R9.1
- new net: R5.2, SW2.2
- new net: R6.1, SW2.3 (K)
- new net led_green: D2.1 (K), R10.1
- new net led_green_2: D1.1 (K), R7.1
- new net led_red: D3.1 (K), R11.1
- new net reg 6v adj: R1.2, R2.1, U3.1 (ADJ)
Other:
- note added: "3.3v logic regulator"
- note added: "6v servo regulator"
- note added: "R2/R1 = 4.8"
- note added: "close to rp2040"
- note added: "important GROUND ALL AROUND THIS"
- note added: "included a led so know when held down"
- note added: "just so we know that the usb-c is powering it"
- note added: "serial wire debug?"
- note added: "so we can switch between battery and usb-c for power"
- note added: "the 1uf caps are on pins 44/45"
- moved on the sheet: U1

Commit message: made a lot of changes, nearly done
Parts:
- removed U6: MPU-6050, Sensor_Motion:InvenSense_QFN-24_4x4mm_P0.5mm, symbol Sensor_Motion:MPU-6050
- added AE?: APAE1575R1540AZDB2F-T, symbol Device:Antenna
- added C? (x4): 10u, symbol Device:C
- added C?: 100n, symbol Device:C
- added C?: 4u7, symbol Device:C
- added C? (x5): 0.1u, symbol Device:C
- added C?: 1u, symbol Device:C
- added C?: 2n2, symbol Device:C
- added C?: 10n, symbol Device:C
- added D?: LED_RED, symbol Device:LED
- added JP?: SolderJumper_2_Bridged, symbol Jumper:SolderJumper_2_Bridged
- added R?: 330, symbol Device:R
- added R? (x4): 2k7, symbol Device:R
- added U?: MPU-6050, Sensor_Motion:InvenSense_QFN-24_4x4mm_P0.5mm, symbol Sensor_Motion:MPU-6050
Connections:
- net 3.3v rail: now also J1.4 (VDD), U5.10 (VDD), U7.13 (VDDIO), U7.2 (VDD), U7.4 (SPI_CS), U8.1 (VCC), U9.22 (V_BCKP), U9.23 (VCC), C?.1, C?.1, C?.1, C?.1, C?.1, C?.1, C?.1, C?.2, C?.2, C?.2, C?.2, JP?.2 (B), R?.2, R?.2, R?.2, R?.2, U?.13 (VDD), U?.8 (VDDIO)
- net GND: now also J1.6 (VSS), J1.9 (SHIELD), U5.3 (GND), U5.5 (SA0/MISO), U5.8 (GND), U5.9 (GND), U7.11 (GND), U7.9 (GND), U8.10 (GND), U8.16 (GND), U8.2 (GND), U8.7 (GND), U9.10 (GND), U9.12 (GND), U9.13 (GND), U9.24 (GND), U9.7 (VDD_USB), C?.1, C?.1, C?.1, C?.1, C?.1, C?.1, C?.1, C?.2, C?.2, C?.2, C?.2, C?.2, C?.2, C?.2, R?.2, U?.18 (GND)
- net ~{CS}: now reaches U5.1 (VDDio)
- net ~{CS}: now also U5.6 (~{CS}), JP?.1 (A)
- net LPS_SCL: now reaches U5.2 (SCL/SCLK)
- net LPS_SDA: now reaches U5.4 (SDA/MOSI)
- net LPS_INT_DRDY: now reaches U5.7 (INT_DRDY)
- net LORA_NRESET: now reaches U8.11 (NRESET)
- net LORA_BUSY: now reaches U8.12 (BUSY)
- net DIO1: now reaches U8.13 (DIO1)
- net DIO2: now reaches U8.14 (DIO2)
- net DIO3: now reaches U8.15 (DIO3)
- net LORA_MISO: now reaches U8.3 (MISO_TX)
- net LORA_MOSI: now reaches U8.4 (MOSI_RX)
- net LORA SCK: now reaches U8.5 (SCK_RTSN)
- net LORA_NSS: now reaches U8.6 (NSS_CTS)
- net LORA_RX_EN: now reaches U8.8 (RX_EN)
- net LORA_TX_EN: now reaches U8.9 (TX_EN)
- net IMU_AUX_SCL: now reaches U7.1 (SCL/SPI_SCK)
- net IMU_AUX_SCL: now also R?.1, U?.7 (AUX_SCL)
- net at U7.10 (CAP): now also C?.2
- net MMC_INT: now reaches U7.15 (INT)
- net IMU_AUX_SDA: now reaches U7.16 (SDA/SPI_SDI)
- net IMU_AUX_SDA: now also R?.1, U?.6 (AUX_SDA)
- net microSD_CS: now reaches J1.2 (DAT3/CD)
- net microSD_MOSI: now reaches J1.3 (CMD)
- net microSD_CLK: now reaches J1.5 (CLK)
- net microSD_MISO: now reaches J1.7 (DAT0)
- net NEO_RF_IN: now reaches U9.11 (RF_IN)
- net NEO_RF_IN: now also AE?.1 (A)
- net NEO_LNA_EN: now reaches U9.14 (LNA_EN)
- net NEO_TXD: now reaches U9.20 (TXD/SPI_MISO)
- net NEO_RXD: now reaches U9.21 (RXD/SPI_MOSI)
- net at U9.3 (TIMEPULSE): now also D?.2 (A)
- net NEO_~{RESET}: now reaches U9.8 (~{RESET})
- net NEO_VCC_RF: now reaches U9.9 (VCC_RF)
- new net: C?.2, C?.2, U?.10 (REGOUT), U?.20 (CPOUT)
- new net IMU_AD0: U?.9 (AD0)
- new net IMU_CLKIN: U?.1 (CLKIN)
- new net IMU_FSYNC: U?.11 (FSYNC)
- new net IMU_INT: U?.12 (INT)
- new net IMU_SCL: R?.1, U?.23 (SCL)
- new net IMU_SDA: R?.1, U?.24 (SDA)
- new net led_red_2: D?.1 (K), R?.1
- no-connect marks 2 -> 12
Other:
- note added: "0.1u for pin 10 2n2 for pin 20"
- note added: "???"
- note added: "RX_EN & TX_EN are for external amps on chip"
- note added: "also 12, 13, 24"
- note added: "busses? who gives a crap about busses???"
- note added: "check whether this decouple is good"
- note added: "do I add an LNA???"
- note added: "dont know what to do with these"
- note added: "i think the shield gets grounded?"
- note added: "idk if VDD_IO is to be pinned high or low???"
- note added: "in SPI mode"
- note added: "lcsc has some 7k of these"
- note added: "messy I know"
- note added: "no idea what to do with interupt pins"
- note added: "not using usb"
- note added: "note: these are sensitive components therefor under both of these is a full ground plane set"
- note added: "one pair for each pin"
- note added: "pin 13"
- note added: "pin 8"
- note added: "pins 9, 8 and 3 are tied to ground???"
- note added: "pullup resistors"
- note added: "the data sheet says to leave open"
- note added: "this is an output, I dont know what it does"
- note added: "ties to ground"
- note added: "todo: add periferals to rp2040"
- note added: "uhhh this may need to become a module???"
- note added: "used for a powered ant"
- note added: "you can add bars :>"
- company: (none) -> Mann co.
- title: (none) -> Engineering 2023 UAV flight controller
- moved on the sheet: U5, U7, U8, U9
