File: Engineering 2023 UAV flight controller/Engineering 2023 UAV flight controller.kicad_sch (KiCad schematic)
At the start: 75 parts, among them J1 Micro_SD_Card, J2 ESC speed control, J3 USB_C_Receptacle_USB2.0, M1 Aileron Left, M2 Aileron Right, M3 Elevator Left, M4 Elevator Right, SW1 SW_SPDT, SW2 SW_Push_LED, U1 W25Q128JVS, U2 AMS1117-3.3, U3 LM350_TO220, U4 RP2040, U5 LPS25HB, U7 MMC5983MA, U8 E28-2G4M27S, U9 NEO-M8N, Y1 ABLS-12.000MHZ-B4-T

Commit message: basicly finished schem, need to finalise the rf ant for the gps
Parts:
- added J?: External pinout, symbol Connector_Generic:Conn_01x10
- added J?: external power rails, symbol Connector_Generic:Conn_02x10_Top_Bottom
- C32: renamed from C?; value 100n -> 0.1u
- SW2: value SW_Push_LED -> 4FSH922
- gave numbers to parts that had none: 22
Connections:
- net IMU_AD0 is gone; now on net GND: U6.9 (AD0)
- net IMU_CLKIN is gone; now on net GND: U6.1 (CLKIN)
- net IMU_FSYNC is gone; now on net GND: U6.11 (FSYNC)
- net LORA_NRESET is gone; now on net 3.3v rail: U8.11 (NRESET)
- net LORA_NSS is gone; now on net LORA_~{SS}: U8.6 (NSS_CTS)
- net LPS_SCL is gone; now on net IMU_SCL: U5.2 (SCL/SCLK)
- net LPS_SDA is gone; now on net IMU_SDA: U5.4 (SDA/MOSI)
- net 3.3v rail: now also SW2.3, J?.1 (Pin_1), J?.10 (Pin_10), J?.2 (Pin_2), J?.3 (Pin_3), J?.4 (Pin_4), J?.5 (Pin_5), J?.6 (Pin_6), J?.7 (Pin_7), J?.8 (Pin_8), J?.9 (Pin_9); no longer SW2.4 (A)
- net Aileron Left PWM: now also U4.38 (GPIO26_ADC0)
- net Aileron Right PWM: now also U4.39 (GPIO27_ADC1)
- net ESC PWM: now also U4.37 (GPIO25)
- net Elevator Left PWM: now also U4.40 (GPIO28_ADC2)
- net Elevator Right PWM: now also U4.41 (GPIO29_ADC3)
- net GND: now also J?.11 (Pin_11), J?.12 (Pin_12), J?.13 (Pin_13), J?.14 (Pin_14), J?.15 (Pin_15), J?.16 (Pin_16), J?.17 (Pin_17), J?.18 (Pin_18), J?.19 (Pin_19), J?.20 (Pin_20); no longer R6.2
- net IMU_SCL: now also U4.5 (GPIO3)
- net IMU_SDA: now also U4.4 (GPIO2)
- net LORA SCK: now also U4.13 (GPIO10)
- net LORA_BUSY: now also U4.15 (GPIO12)
- net LORA_MISO: now also U4.11 (GPIO8)
- net LORA_MOSI: now also U4.14 (GPIO11)
- net LORA_RX_EN: now also U4.35 (GPIO23)
- net LORA_TX_EN: now also U4.36 (GPIO24)
- net NEO_RXD: now also U4.2 (GPIO0)
- net NEO_TXD: now also U4.3 (GPIO1)
- net microSD_CLK: now also U4.8 (GPIO6)
- net microSD_CS: now also U4.7 (GPIO5)
- net microSD_MISO: now also U4.6 (GPIO4)
- net microSD_MOSI: now also U4.9 (GPIO7)
- net sw_led: now reaches SW2.2
- net sw_led: now also R6.2; no longer R5.2
- net sw_r: now reaches R6.1
- net sw_r: now also R5.2, SW2.4; no longer SW2.3 (K)
- net LORA_~{SS}: now reaches U4.12 (GPIO9)
- net External_pin_1: now reaches U4.16 (GPIO13)
- net External_pin_1: now also J?.1 (Pin_1)
- net External_pin_2: now reaches U4.17 (GPIO14)
- net External_pin_2: now also J?.2 (Pin_2)
- net External_pin_3: now reaches U4.18 (GPIO15)
- net External_pin_3: now also J?.3 (Pin_3)
- net External_pin_4: now reaches U4.27 (GPIO16)
- net External_pin_4: now also J?.4 (Pin_4)
- net External_pin_5: now reaches U4.28 (GPIO17)
- net External_pin_5: now also J?.5 (Pin_5)
- net External_pin_6: now reaches U4.29 (GPIO18)
- net External_pin_6: now also J?.6 (Pin_6)
- net External_pin_7: now reaches U4.30 (GPIO19)
- net External_pin_7: now also J?.7 (Pin_7)
- net External_pin_8: now reaches U4.31 (GPIO20)
- net External_pin_8: now also J?.8 (Pin_8)
- net External_pin_9: now reaches U4.32 (GPIO21)
- net External_pin_9: now also J?.9 (Pin_9)
- net External_pin_10: now reaches U4.34 (GPIO22)
Other:
- note added: "External pinout"
- note added: "I^{2}C1 SDA and SCL"
- note added: "SPI0 line"
- note added: "SPI1 line"
- note added: "Uart0 TX and RX"
- note added: "close together"
- note added: "gonna bus these two"
- note added: "idk what to do with these two???"
- note added: "need to decide on rf ant stuff before pcb can be designed"
- note added: "not using the DIO"
- note added: "note that these two do have addresses"
- note added: "pins 13 to 22 on rp2040"
- note added: "pulling the ~{RESET} high to prevent it reseting"
- note added: "these last five are hooked up to pwm"
- note added: "to tell if lora module is busy"
- note added: "will be using the pio to connect with these"
- note removed: "do I add an LNA???"
- moved on the sheet: R6
