File: Engineering 2023 UAV flight controller/Engineering 2023 UAV flight controller.kicad_sch (KiCad schematic)
At the start: 103 parts, among them IC1 LM2577SX-ADJ_NOPB, J1 Micro_SD_Card, J10 DIO, J2 ESC speed control, J3 USB_C_Receptacle_USB2.0, J4 Conn_Coaxial, J5 external power rail, J6 GPIO, J7 external ground rail, J8 Serial wire debug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

Commit message: aaaaa
Parts:
- IC1: footprint Package_TO_SOT_THT:TO-220-5_Horizontal_TabDown -> Package_TO_SOT_SMD:TO-263-5_TabPin3
Connections:
- net FEEDBACK: now reaches IC1.2 (FEEDBACK), R2.2, R20.1
- net L-D: now reaches D5.2 (A), IC1.4 (SWITCH), L2.2
Changed lines of the file:
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@@
     (effects (font (size 1.27 1.27)) (justify right bottom))
   )
+  (label "SWITCH" (at 124.46 31.75 0)
+    (effects (font (size 1.27 1.27)) (justify left bottom))
+  )
   (label "QSPI_SS" (at 83.82 207.01 0)
     (effects (font (size 1.27 1.27)) (justify left bottom))
@@
     (effects (font (size 1.27 1.27)) (justify left bottom))
   )
+  (label "L-D" (at 114.3 20.32 0)
+    (effects (font (size 1.27 1.27)) (justify left bottom))
+  )
   (label "LPS_INT_DRDY" (at 215.9 49.53 180)
     (effects (font (size 1.27 1.27)) (justify right bottom))
@@
     (effects (font (size 1.27 1.27)) (justify left bottom))
   )
+  (label "FEEDBACK" (at 132.08 35.56 180)
+    (effects (font (size 1.27 1.27)) (justify right bottom))
+  )
   (label "QSPI_SCLK" (at 22.86 219.71 0)
     (effects (font (size 1.27 1.27)) (justify left bottom))
@@
     (property "Reference" "IC1" (id 0) (at 106.68 24.13 0))
     (property "Value" "LM2577SX-ADJ_NOPB" (id 1) (at 106.68 26.67 0))
-    (property "Footprint" "Package_TO_SOT_THT:TO-220-5_Horizontal_TabDown" (id 2) (at 137.16 34.29 0)
+    (property "Footprint" "Package_TO_SOT_SMD:TO-263-5_TabPin3" (id 2) (at 137.16 34.29 0)
       (effects (font (size 1.27 1.27)) (justify left) hide)
     )
@@
     )
     (path "/406cb148-776b-4495-8741-9c38334f3acd"
-      (reference "IC1") (unit 1) (value "LM2577SX-ADJ_NOPB") (footprint "Package_TO_SOT_THT:TO-220-5_Horizontal_TabDown")
+      (reference "IC1") (unit 1) (value "LM2577SX-ADJ_NOPB") (footprint "Package_TO_SOT_SMD:TO-263-5_TabPin3")
     )
     (path "/b831070f-41fa-4fff-9268-47aed16ea16b"

Commit message: revision 2 complete, need to upload for review
Parts:
- C38: footprint Capacitor_SMD:C_0603_1608Metric -> Capacitor_SMD:CP_Elec_5x3
Changed lines of the file:
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@@
     (property "Reference" "C38" (id 0) (at 370.84 83.82 90))
     (property "Value" "47u" (id 1) (at 375.92 80.01 90))
-    (property "Footprint" "Capacitor_SMD:C_0603_1608Metric" (id 2) (at 375.92 82.55 0)
+    (property "Footprint" "Capacitor_SMD:CP_Elec_5x3" (id 2) (at 375.92 82.55 0)
       (effects (font (size 1.27 1.27)) hide)
     )
@@
     )
     (path "/cba63941-61fa-4b4b-9985-1ec80e22491b"
-      (reference "C38") (unit 1) (value "47u") (footprint "Capacitor_SMD:C_0603_1608Metric")
+      (reference "C38") (unit 1) (value "47u") (footprint "Capacitor_SMD:CP_Elec_5x3")
     )
     (path "/f1ac7a2c-9d99-4f4c-8436-c84f3d4531ff"

Commit message: revision 2 complete, need to upload for review sent off rev 2 for review
Parts:
- added H1, H2, H3, H4: MountingHole_Pad, MountingHole:MountingHole_3.2mm_M3_Pad_Via, symbol Mechanical:MountingHole_Pad
Connections:
- net GND: now also H1.1, H2.1, H3.1, H4.1
Changed lines of the file:
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@@
   (junction (at 77.47 110.49) (diameter 0) (color 0 0 0 0)
   )
+  (junction (at 391.16 248.92) (diameter 0) (color 0 0 0 0)
+  )
   (junction (at 232.41 110.49) (diameter 0) (color 0 0 0 0)
   )
@@
   (junction (at 104.14 124.46) (diameter 0) (color 0 0 0 0)
   )
+  (junction (at 388.62 248.92) (diameter 0) (color 0 0 0 0)
+  )
   (junction (at 256.54 86.36) (diameter 0) (color 0 0 0 0)
   )
@@
   (junction (at 57.15 261.62) (diameter 0) (color 0 0 0 0)
   )
+  (junction (at 393.7 248.92) (diameter 0) (color 0 0 0 0)
+  )
   (junction (at 367.03 97.79) (diameter 0) (color 0 0 0 0)
   )
@@
     (stroke (width 0) (type default) (color 0 0 0 0))
   )
+  (wire (pts (xy 391.16 248.92) (xy 393.7 248.92))
+    (stroke (width 0) (type default) (color 0 0 0 0))
+  )
   (wire (pts (xy 228.6 209.55) (xy 240.03 209.55))
     (stroke (width 0) (type default) (color 0 0 0 0))
@@
     (stroke (width 0) (type default) (color 0 0 0 0))
   )
+  (wire (pts (xy 393.7 248.92) (xy 398.78 248.92))
+    (stroke (width 0) (type default) (color 0 0 0 0))
+  )
   (wire (pts (xy 270.51 176.53) (xy 285.75 176.53))
     (stroke (width 0) (type default) (color 0 0 0 0))
@@
     (stroke (width 0) (type default) (color 0 0 0 0))
   )
+  (wire (pts (xy 383.54 248.92) (xy 388.62 248.92))
+    (stroke (width 0) (type default) (color 0 0 0 0))
+  )
   (wire (pts (xy 382.27 195.58) (xy 382.27 198.12))
     (stroke (width 0) (type default) (color 0 0 0 0))
@@
     (stroke (width 0) (type default) (color 0 0 0 0))
   )
+  (wire (pts (xy 388.62 248.92) (xy 391.16 248.92))
+    (stroke (width 0) (type default) (color 0 0 0 0))
+  )
   (wire (pts (xy 252.73 193.04) (xy 254 193.04))
     (stroke (width 0) (type default) (color 0 0 0 0))
@@
     (stroke (width 0) (type default) (color 0 0 0 0))
   )
+  (wire (pts (xy 391.16 250.19) (xy 391.16 248.92))
+    (stroke (width 0) (type default) (color 0 0 0 0))
+  )
   (wire (pts (xy 264.16 91.44) (xy 264.16 73.66))
     (stroke (width 0) (type default) (color 0 0 0 0))
@@
     (pin "1")
   )
+  (symbol (lib_id "Mechanical:MountingHole_Pad") (at 388.62 246.38 0) (unit 1)
+    (in_bom yes) (on_board yes) (fields_autoplaced)
+    (property "Reference" "H2" (id 0) (at 391.16 243.8399 0)
+      (effects (font (size 1.27 1.27)) (justify left))
+    )
+    (property "Value" "MountingHole_Pad" (id 1) (at 391.16 246.3799 0)
+      (effects (font (size 1.27 1.27)) (justify left) hide)
+    )
+    (property "Footprint" "MountingHole:MountingHole_3.2mm_M3_Pad_Via" (id 2) (at 388.62 246.38 0)
+      (effects (font (size 1.27 1.27)) hide)
+    )
+    (property "Datasheet" "~" (id 3) (at 388.62 246.38 0)
+      (effects (font (size 1.27 1.27)) hide)
+    )
+    (pin "1")
+  )
   (symbol (lib_id "Sensor_Pressure:LPS25HB") (at 185.42 41.91 0) (unit 1)
     (in_bom yes) (on_board yes) (fields_autoplaced)
@@
     (pin "3")
   )
+  (symbol (lib_id "power:GND") (at 391.16 250.19 0) (unit 1)
+    (in_bom yes) (on_board yes)
+    (property "Reference" "#PWR08" (id 0) (at 391.16 256.54 0)
+      (effects (font (size 1.27 1.27)) hide)
+    )
+    (property "Value" "GND" (id 1) (at 394.97 251.46 0))
+    (property "Footprint" "" (id 2) (at 391.16 250.19 0)
+      (effects (font (size 1.27 1.27)) hide)
+    )
+    (property "Datasheet" "" (id 3) (at 391.16 250.19 0)
+      (effects (font (size 1.27 1.27)) hide)
+    )
+    (pin "1")
+  )
   (symbol (lib_id "power:GND") (at 302.26 179.07 0) (unit 1)
     (in_bom yes) (on_board yes) (fields_autoplaced)
@@
     (pin "2")
   )
+  (symbol (lib_id "Mechanical:MountingHole_Pad") (at 398.78 246.38 0) (unit 1)
+    (in_bom yes) (on_board yes) (fields_autoplaced)
+    (property "Reference" "H4" (id 0) (at 401.32 243.8399 0)
+      (effects (font (size 1.27 1.27)) (justify left))
+    )
+    (property "Value" "MountingHole_Pad" (id 1) (at 401.32 246.3799 0)
+      (effects (font (size 1.27 1.27)) (justify left) hide)
+    )
+    (property "Footprint" "MountingHole:MountingHole_3.2mm_M3_Pad_Via" (id 2) (at 398.78 246.38 0)
+      (effects (font (size 1.27 1.27)) hide)
+    )
+    (property "Datasheet" "~" (id 3) (at 398.78 246.38 0)
+      (effects (font (size 1.27 1.27)) hide)
+    )
+    (pin "1")
+  )
   (symbol (lib_id "power:GND") (at 232.41 113.03 0) (unit 1)
     (in_bom yes) (on_board yes)
@@
     (pin "2")
   )
+  (symbol (lib_id "Mechanical:MountingHole_Pad") (at 393.7 246.38 0) (unit 1)
+    (in_bom yes) (on_board yes) (fields_autoplaced)
+    (property "Reference" "H3" (id 0) (at 396.24 243.8399 0)
+      (effects (font (size 1.27 1.27)) (justify left))
+    )
+    (property "Value" "MountingHole_Pad" (id 1) (at 396.24 246.3799 0)
+      (effects (font (size 1.27 1.27)) (justify left) hide)
+    )
+    (property "Footprint" "MountingHole:MountingHole_3.2mm_M3_Pad_Via" (id 2) (at 393.7 246.38 0)
+      (effects (font (size 1.27 1.27)) hide)
+    )
+    (property "Datasheet" "~" (id 3) (at 393.7 246.38 0)
+      (effects (font (size 1.27 1.27)) hide)
+    )
+    (pin "1")
+  )
   (symbol (lib_id "Memory_Flash:W25Q128JVS") (at 45.72 217.17 0) (unit 1)
     (in_bom yes) (on_board yes) (fields_autoplaced)
@@
     (pin "9")
   )
+  (symbol (lib_id "Mechanical:MountingHole_Pad") (at 383.54 246.38 0) (unit 1)
+    (in_bom yes) (on_board yes)
+    (property "Reference" "H1" (id 0) (at 386.08 243.8399 0)
+      (effects (font (size 1.27 1.27)) (justify left))
+    )
+    (property "Value" "MountingHole_Pad" (id 1) (at 383.54 241.3 0)
+      (effects (font (size 1.27 1.27)) (justify left))
+    )
+    (property "Footprint" "MountingHole:MountingHole_3.2mm_M3_Pad_Via" (id 2) (at 383.54 246.38 0)
+      (effects (font (size 1.27 1.27)) hide)
+    )
+    (property "Datasheet" "~" (id 3) (at 383.54 246.38 0)
+      (effects (font (size 1.27 1.27)) hide)
+    )
+    (pin "1")
+  )
   (symbol (lib_id "Graphic:SYM_Radio_Waves_Large") (at 254 276.86 0) (unit 1)
     (in_bom yes) (on_board yes) (fields_autoplaced)
@@
       (reference "#PWR07") (unit 1) (value "GND") (footprint "")
     )
+    (path "/1b208ee0-2e4b-4eb6-bf1e-e84e13c9bb82"
+      (reference "#PWR08") (unit 1) (value "GND") (footprint "")
+    )
     (path "/dab67dfc-3798-450d-aa72-255b201c5bf6"
       (reference "#PWR09") (unit 1) (value "GND") (footprint "")
@@
       (reference "FB2") (unit 1) (value " BLM15HD102SN1") (footprint "Inductor_SMD:L_0402_1005Metric_Pad0.77x0.64mm_HandSolder")
     )
+    (path "/f595217f-213b-47ee-8de5-450b11e7d9a2"
+      (reference "H1") (unit 1) (value "MountingHole_Pad") (footprint "MountingHole:MountingHole_3.2mm_M3_Pad_Via")
+    )
+    (path "/07889ad4-45c3-4f97-b038-e1b4d20b2a0a"
+      (reference "H2") (unit 1) (value "MountingHole_Pad") (footprint "MountingHole:MountingHole_3.2mm_M3_Pad_Via")
+    )
+    (path "/ca4151f2-1f25-419e-9d28-f56e4e726493"
+      (reference "H3") (unit 1) (value "MountingHole_Pad") (footprint "MountingHole:MountingHole_3.2mm_M3_Pad_Via")
+    )
+    (path "/6cf3cf31-7265-4259-8d35-548d1e6b2422"
+      (reference "H4") (unit 1) (value "MountingHole_Pad") (footprint "MountingHole:MountingHole_3.2mm_M3_Pad_Via")
+    )
     (path "/406cb148-776b-4495-8741-9c38334f3acd"
