File: Engineering 2023 UAV flight controller/Engineering 2023 UAV flight controller.kicad_pcb (KiCad board)
At the start: 4 copper layers, 72.7 x 100 mm, 73 parts, among them J1 Micro_SD_Card, J10 DIO, J3 USB_C_Receptacle_USB2.0, J4 Conn_Coaxial, J5 external power rail, J6 GPIO, J7 external ground rail, J8 Serial wire debug, J9 reset short?, M1 Aileron Left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

Commit message: started layout for the power part of board, addded some beads to NEO RX/TX
Parts:
- added C1: 0.1uf, Capacitor_SMD:C_0603_1608Metric, F.Cu at (255.0, 113.6)
- added C2: 0.1uf, Capacitor_SMD:C_0603_1608Metric, F.Cu at (87.6, 139.0)
- added C3: 1uf, Capacitor_SMD:C_0603_1608Metric, F.Cu at (241.7, 128.5)
- added C38: 47u, Capacitor_SMD:C_0603_1608Metric, F.Cu at (245.7, 125.9)
- added C39: 2u2, Capacitor_SMD:C_0603_1608Metric, F.Cu at (151.8, 59.8)
- added C4: 0.1uf, Capacitor_SMD:C_0603_1608Metric, F.Cu at (241.7, 126.0)
- added C40: 4u7, Capacitor_SMD:C_0603_1608Metric, F.Cu at (159.8, 61.0)
- added C41: 2u2, Capacitor_SMD:C_0603_1608Metric, F.Cu at (158.6, 57.2)
- added C5: 0.33u, Capacitor_SMD:C_0603_1608Metric, F.Cu at (84.6, 140.6)
- added C6: 680u, Capacitor_SMD:C_0603_1608Metric, F.Cu at (95.4, 143.0)
- added D2: LED_GREEN, LED_SMD:LED_0603_1608Metric, F.Cu at (239.4, 123.4)
- added D3: LED_RED, LED_SMD:LED_0603_1608Metric, F.Cu at (88.2, 147.4)
- added D5: D_Schottky, Diode_SMD:D_SMA, F.Cu at (94.2, 149.6)
- added FB1: BLM15HD102SN1, Inductor_SMD:L_0402_1005Metric_Pad0.77x0.64mm_HandSolder, F.Cu at (216.2, 139.8)
- added FB2: BLM15HD102SN1, Inductor_SMD:L_0402_1005Metric_Pad0.77x0.64mm_HandSolder, F.Cu at (212.9, 139.8)
- added IC1: LM2577SX-ADJ_NOPB, Package_TO_SOT_THT:TO-220-5_Horizontal_TabDown, F.Cu at (90.4, 133.2)
- added J2: ESC speed control, Connector_PinHeader_2.54mm:PinHeader_1x03_P2.54mm_Vertical, F.Cu at (181.1, 120.0)
- added L2: 100u, Inductor_SMD:L_Wuerth_WE-PD-Typ-LS, F.Cu at (101.6, 154.8)
- added R1: 2k2, Resistor_SMD:R_0603_1608Metric, F.Cu at (76.6, 141.0)
- added R10: 330, Resistor_SMD:R_0603_1608Metric, F.Cu at (250.4, 120.7)
- added R11: 330, Resistor_SMD:R_0603_1608Metric, F.Cu at (78.6, 146.0)
- added R2: 1K2, Resistor_SMD:R_0603_1608Metric, F.Cu at (80.2, 150.6)
- added R20: 330, Resistor_SMD:R_0603_1608Metric, F.Cu at (90.0, 140.8)
- added R21: 330, Resistor_SMD:R_0603_1608Metric, F.Cu at (161.8, 59.0)
- added SW1: SW_SPDT, Button_Switch_SMD:SW_SPDT_CK-JS102011SAQN, F.Cu at (186.2, 128.0)
- added TP1: 6v tp, TestPoint:TestPoint_Pad_D2.5mm, F.Cu at (227.2, 136.7)
- added TP2: 3.3 tp, TestPoint:TestPoint_Pad_D2.5mm, F.Cu at (250.7, 114.6)
- added TP3: NEO 3.3 tp, TestPoint:TestPoint_Pad_D2.5mm, F.Cu at (203.6, 53.8)
- added U2: NCP1117-3.3_TO252, Package_TO_SOT_SMD:TO-252-2, F.Cu at (228.9, 130.4)
- added U3: LP2987-3.3_WSON8, Package_SON:WSON-8-1EP_4x4mm_P0.8mm_EP2.2x3mm, F.Cu at (155.4, 59.4)
- moved J8 49.1 mm to (145.0, 111.9)
- moved J9 49.1 mm to (145.0, 105.9)
- moved C23 0.20 mm to (165.6, 56.6)
Connections:
- C23 pad 1: /3.3v rail -> /NEO 3.3v rail
- C26 pad 1: /3.3v rail -> /NEO 3.3v rail
- C28 pad 1: /3.3v rail -> /NEO 3.3v rail
- C29 pad 1: /3.3v rail -> /NEO 3.3v rail
- U9 pad 20: /NEO_TXD -> /NEO_FB_TXD
- U9 pad 21: /NEO_RXD -> /NEO_FB_RXD
- U9 pad 22: /3.3v rail -> /NEO 3.3v rail
- U9 pad 23: /3.3v rail -> /NEO 3.3v rail
Routing:
- net /NEO_TXD: track 82.4 -> 0.00 mm, vias 2 -> 0
- net /NEO_FB_TXD: track 0.00 -> 82.4 mm, vias 0 -> 2
- net /NEO_RXD: track 82.2 -> 0.00 mm, vias 2 -> 0
- net /NEO_FB_RXD: track 0.00 -> 82.2 mm, vias 0 -> 2
- net /NEO 3.3v rail: track 0.00 -> 23.9 mm
- net /3.3v rail: track 109.8 -> 87.9 mm, vias 27 -> 25
- net /~{LDO_ERROR}: track 0.00 -> 5.09 mm

Commit message: aaaaa
Parts:
- IC1: footprint Package_TO_SOT_THT:TO-220-5_Horizontal_TabDown -> Package_TO_SOT_SMD:TO-263-5_TabPin3
- TP3: moved to B.Cu
- moved R1 69.9 mm to (145.2, 127.8), turned to -90 degrees
- moved R2 67.5 mm to (140.4, 120.0)
- moved C5 61.4 mm to (145.2, 131.0), turned to -90 degrees
- moved R20 53.9 mm to (140.4, 121.6), turned to 180 degrees
- moved R11 52.3 mm to (119.0, 112.8), turned to 180 degrees
- moved D3 48.6 mm to (122.4, 112.8)
- moved IC1 48.2 mm to (138.6, 132.6), turned to -90 degrees
- moved D5 48.0 mm to (132.2, 120.2), turned to -90 degrees
- moved C6 46.3 mm to (135.0, 119.0), turned to 90 degrees
- moved C2 45.3 mm to (132.0, 129.8), turned to -90 degrees
- moved L2 38.0 mm to (123.8, 124.0), turned to 90 degrees
- moved TP3 27.0 mm to (176.8, 57.2), turned to 180 degrees
Connections:
- net Net-(D5-Pad2) renamed /L-D
- net Net-(IC1-Pad2) renamed /FEEDBACK
Routing:
- net /NEO 3.3v rail: track 23.9 -> 31.3 mm, vias 0 -> 1
- net GND: track 68.3 -> 73.1 mm, vias 94 -> 101
- net /reg in: track 0.00 -> 3.60 mm
- net /Servo 6V rail: track 11.0 -> 13.8 mm
- net Net-(D3-Pad1): track 0.00 -> 1.79 mm
- added copper zone on F.Cu, net /L-D
- added copper zone on F.Cu, net /Servo 6V rail
- added copper zone on F.Cu, net /reg in

Commit message: revision 2 complete, need to upload for review
Parts:
- C38: footprint Capacitor_SMD:C_0603_1608Metric -> Capacitor_SMD:CP_Elec_5x3
- moved C38 112.3 mm to (134.2, 112.2)
- moved TP1 102.2 mm to (127.8, 113.0)
- moved R10 96.1 mm to (154.4, 124.2), turned to 180 degrees
- moved C1 94.3 mm to (163.3, 135.6), turned to 180 degrees
- moved FB1 85.8 mm to (178.4, 62.8), turned to 180 degrees
- moved FB2 85.5 mm to (178.4, 61.6), turned to 180 degrees
- moved D2 81.6 mm to (157.8, 124.2)
- moved TP2 81.3 mm to (170.2, 125.8)
- moved C3 79.5 mm to (162.5, 121.8), turned to 90 degrees
- moved C4 77.5 mm to (164.3, 121.8), turned to 90 degrees
- moved U2 65.7 mm to (163.3, 129.0), turned to 90 degrees
- moved J8 37.4 mm to (137.0, 75.4), turned to 0 degrees
- moved J9 30.3 mm to (133.2, 78.0), turned to 180 degrees
- moved TP3 21.4 mm to (156.4, 63.8)
- moved C2 1.43 mm to (132.0, 128.3)
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Routing:
- net /reg in: track 3.60 -> 100.5 mm, vias 0 -> 12
- net /NEO_TXD: track 0.00 -> 72.9 mm, vias 0 -> 2
- net /NEO_FB_RXD: track 82.2 -> 11.5 mm, vias 2 -> 0
- net /NEO_FB_TXD: track 82.4 -> 13.0 mm
- net /NEO_RXD: track 0.00 -> 68.8 mm, vias 0 -> 2
- net /ESC PWM: track 9.05 -> 71.4 mm
- net GND: track 73.1 -> 106.2 mm, vias 101 -> 115
- net /USB_C positive rail: track 21.9 -> 52.4 mm, vias 0 -> 2
- net /SWCLK: track 3.61 -> 23.2 mm, vias 1 -> 0
- net /RUN: track 5.06 -> 23.7 mm
- net /3.3v rail: track 87.9 -> 103.0 mm, vias 25 -> 34
- net /SWD: track 6.91 -> 20.4 mm
- net /FEEDBACK: track 0.00 -> 7.21 mm
- net /Servo 6V rail: track 13.8 -> 20.0 mm
- net Net-(IC1-Pad1): track 0.00 -> 3.26 mm
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- added copper zone on F.Cu, net /ESC positive rail
- added copper zone on In2.Cu, net /reg in
Other:
- board text removed: "TODO: reroute pcb to add space at power zone for a switching regulator, add tabs for pcb mounting"

Commit message: revision 2 complete, need to upload for review sent off rev 2 for review
Parts:
- added H1: MountingHole_Pad, MountingHole:MountingHole_3.2mm_M3_Pad_Via, F.Cu at (109.4, 136.0)
- added H2: MountingHole_Pad, MountingHole:MountingHole_3.2mm_M3_Pad_Via, F.Cu at (194.2, 48.0)
- added H3: MountingHole_Pad, MountingHole:MountingHole_3.2mm_M3_Pad_Via, F.Cu at (194.2, 136.0)
- added H4: MountingHole_Pad, MountingHole:MountingHole_3.2mm_M3_Pad_Via, F.Cu at (109.4, 48.0)
Routing:
- net GND: vias 115 -> 119
Other:
- board size 72.7 x 100 mm -> 96.9 x 100 mm

Commit message: changes
Routing:
- net /Servo 6V rail: track 20.0 -> 9.01 mm
Changed lines of the file:
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@@
   (segment (start 139.2 116.775) (end 135.025 116.775) (width 0.3) (layer "F.Cu") (net 3))
   (segment (start 135.025 116.775) (end 135 116.8) (width 0.3) (layer "F.Cu") (net 3))
-  (segment (start 121.66 108.4) (end 121.66 97.425) (width 0.3) (layer "F.Cu") (net 3))
   (segment (start 132.225 116.8) (end 132.2 116.775) (width 0.3) (layer "F.Cu") (net 3))
   (segment (start 139.575 117.15) (end 139.2 116.775) (width 0.3) (layer "F.Cu") (net 3))

Commit message: more stuff done
Parts:
- C6: footprint Capacitor_SMD:C_0603_1608Metric -> Capacitor_SMD:CP_Elec_8x6.5
- moved C6 9.30 mm to (144.2, 116.2)
- moved R2 8.69 mm to (148.2, 122.4)
- moved R20 8.66 mm to (148.2, 124.0)
Connections:
- C6 pad 1: GND -> /Servo 6V rail
- C6 pad 2: /Servo 6V rail -> GND
Routing:
- net /Servo 6V rail: track 9.01 -> 0.07 mm
- net /ESC PWM: track 71.4 -> 63.9 mm
- net GND: track 106.2 -> 101.9 mm, vias 119 -> 118
- net /FEEDBACK: track 7.21 -> 3.12 mm
- net /Elevator Right PWM: track 36.6 -> 35.5 mm

Commit message: .
Parts:
- moved R20 8.85 mm to (139.6, 121.8)
- moved R2 7.21 mm to (141.4, 120.0), turned to 180 degrees
- moved C6 2.95 mm to (142.8, 113.6)
Routing:
- net /Servo 6V rail: track 0.07 -> 14.3 mm
- net GND: track 101.9 -> 106.8 mm
- net /FEEDBACK: track 3.12 -> 4.99 mm
Changed lines of the file:
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@@
   )
   (footprint "Resistor_SMD:R_0603_1608Metric" (layer "F.Cu")
-    (at 148.2 122.4)
+    (at 141.4 120 180)
     (descr "Resistor SMD 0603 (1608 Metric), square (rectangular) end terminal, IPC_7351 nominal, (Body size source: IPC-SM-782 page 72, https://www.pcb-3d.com/wordpress/wp-content/uploads/ipc-sm-782a_amendment_1_and_2.pdf), generated with kicad-footprint-generator")
     (tags "resistor")
@@
     (property "Sheetname" "")
     (attr smd)
-    (fp_text reference "R2" (at 0 -1.43) (layer "F.SilkS")
+    (fp_text reference "R2" (at -2.6 0) (layer "F.SilkS")
       (effects (font (size 1 1) (thickness 0.15)))
     )
@@
     (fp_line (start -0.8 -0.4125) (end 0.8 -0.4125) (layer "F.Fab") (width 0.1))
     (fp_line (start 0.8 0.4125) (end -0.8 0.4125) (layer "F.Fab") (width 0.1))
-    (pad "1" smd roundrect (at -0.825 0) (size 0.8 0.95) (layers "F.Cu" "F.Paste" "F.Mask") (roundrect_rratio 0.25)
+    (pad "1" smd roundrect (at -0.825 0 180) (size 0.8 0.95) (layers "F.Cu" "F.Paste" "F.Mask") (roundrect_rratio 0.25)
       (net 3 "/Servo 6V rail") (pintype "passive"))
-    (pad "2" smd roundrect (at 0.825 0) (size 0.8 0.95) (layers "F.Cu" "F.Paste" "F.Mask") (roundrect_rratio 0.25)
+    (pad "2" smd roundrect (at 0.825 0 180) (size 0.8 0.95) (layers "F.Cu" "F.Paste" "F.Mask") (roundrect_rratio 0.25)
       (net 117 "/FEEDBACK") (pintype "passive"))
     (model "${KICAD6_3DMODEL_DIR}/Resistor_SMD.3dshapes/R_0603_1608Metric.wrl"
@@
   )
   (footprint "Resistor_SMD:R_0603_1608Metric" (layer "F.Cu")
-    (at 148.175 124 180)
+    (at 139.6 121.8 180)
     (descr "Resistor SMD 0603 (1608 Metric), square (rectangular) end terminal, IPC_7351 nominal, (Body size source: IPC-SM-782 page 72, https://www.pcb-3d.com/wordpress/wp-content/uploads/ipc-sm-782a_amendment_1_and_2.pdf), generated with kicad-footprint-generator")
     (tags "resistor")
@@
     (property "Sheetname" "")
     (attr smd)
-    (fp_text reference "R20" (at 0 -1.43) (layer "F.SilkS")
+    (fp_text reference "R20" (at -3 0) (layer "F.SilkS")
       (effects (font (size 1 1) (thickness 0.15)))
     )
@@
   )
   (footprint "Capacitor_SMD:CP_Elec_8x6.5" (layer "F.Cu")
-    (at 144.2 116.2 90)
+    (at 142.8 113.6 90)
     (descr "SMD capacitor, aluminum electrolytic, Rubycon, 8.0x6.5mm")
     (tags "capacitor electrolytic")
@@
     (fp_line (start -3.5 3.5) (end -3.5 -2.5) (layer "F.Fab") (width 0.1))
     (fp_line (start -2.5 -3.5) (end 3.5 -3.5) (layer "F.Fab") (width 0.1))
-    (pad "" smd roundrect locked (at 0.8 -0.8 180) (size 1.29 1.29) (layers "F.Paste") (roundrect_rratio 0.193798))
-    (pad "" smd roundrect locked (at -0.8 0.8 180) (size 1.29 1.29) (layers "F.Paste") (roundrect_rratio 0.193798))
-    (pad "" smd roundrect locked (at 0.8 0.8 180) (size 1.29 1.29) (layers "F.Paste") (roundrect_rratio 0.193798))
-    (pad "" smd roundrect locked (at -0.8 -0.8 180) (size 1.29 1.29) (layers "F.Paste") (roundrect_rratio 0.193798))
+    (pad "" smd roundrect locked (at 0.8 -0.8 180) (size 1.29 1.29) (layers "F.Paste") (roundrect_rratio 0.1937976744))
+    (pad "" smd roundrect locked (at -0.8 0.8 180) (size 1.29 1.29) (layers "F.Paste") (roundrect_rratio 0.1937976744))
+    (pad "" smd roundrect locked (at 0.8 0.8 180) (size 1.29 1.29) (layers "F.Paste") (roundrect_rratio 0.1937976744))
+    (pad "" smd roundrect locked (at -0.8 -0.8 180) (size 1.29 1.29) (layers "F.Paste") (roundrect_rratio 0.1937976744))
     (pad "1" smd roundrect locked (at -3.4375 -2.6 180) (size 0.875 0.2) (layers "F.Cu" "F.Paste" "F.Mask") (roundrect_rratio 0.25)
       (net 2 "/3.3v rail") (pinfunction "IOVDD") (pintype "power_in"))
@@
   (segment (start 165.95 70.225) (end 167.125 70.225) (width 0.3) (layer "F.Cu") (net 1))
   (segment (start 158.05 102.35) (end 157.5 102.35) (width 0.3) (layer "F.Cu") (net 1))
+  (segment (start 138.6 112.2) (end 141.15 112.2) (width 1) (layer "F.Cu") (net 1))
   (segment (start 181.075 107.5) (end 181.075 106.655) (width 0.3) (layer "F.Cu") (net 1))
   (segment (start 118.175 112.8) (end 118.175 109.345) (width 0.3) (layer "F.Cu") (net 1))
   (segment (start 180.825 72.299999) (end 182 72.299999) (width 0.3) (layer "F.Cu") (net 1))
   (segment (start 175.05 113.85) (end 173.875 113.85) (width 0.3) (layer "F.Cu") (net 1))
+  (segment (start 141.15 112.2) (end 142.8 110.55) (width 1) (layer "F.Cu") (net 1))
   (segment (start 165.775 82.35) (end 165.775 81.325) (width 0.3) (layer "F.Cu") (net 1))
   (segment (start 175.6 86.505) (end 175.6 88.05) (width 0.3) (layer "F.Cu") (net 1))
@@
   (segment (start 141.8 63) (end 141.8 65.6) (width 0.3) (layer "In2.Cu") (net 2))
   (segment (start 121.66 97.425) (end 121.685 97.4) (width 0.3) (layer "F.Cu") (net 3))
+  (segment (start 142.225 120) (end 142.225 117.225) (width 0.3) (layer "F.Cu") (net 3))
+  (segment (start 142.675 116.775) (end 142.8 116.65) (width 0.3) (layer "F.Cu") (net 3))
+  (segment (start 142.225 117.225) (end 142.8 116.65) (width 0.3) (layer "F.Cu") (net 3))
+  (segment (start 132.2 116.775) (end 142.675 116.775) (width 1) (layer "F.Cu") (net 3))
   (segment (start 132.225 116.8) (end 132.2 116.775) (width 0.3) (layer "F.Cu") (net 3))
   (segment (start 152.58 87.9325) (end 152.58 82.57) (width 0.25) (layer "F.Cu") (net 4))
@@
   (segment (start 145.05 125.4) (end 145.2 125.55) (width 0.25) (layer "F.Cu") (net 116))
   (segment (start 142 125.4) (end 145.05 125.4) (width 0.25) (layer "F.Cu") (net 116))
+  (segment (start 140.575 121.65) (end 140.425 121.8) (width 0.25) (layer "F.Cu") (net 117))
   (segment (start 140.3 122.275) (end 140.3 125.4) (width 0.25) (layer "F.Cu") (net 117))
+  (segment (start 140.575 120) (end 140.575 121.65) (width 0.25) (layer "F.Cu") (net 117))
   (segment (start 159.8 59) (end 160.625 58.175) (width 0.25) (layer "F.Cu") (net 120))
   (segment (start 157.05 59) (end 159.8 59) (width 0.25) (layer "F.Cu") (net 120))

Commit message: rightio, take two on the pcb.
Parts:
- removed J9: reset short?, Connector_PinHeader_2.54mm:PinHeader_1x02_P2.54mm_Vertical
- removed SW2: 4FSH922, Button_Switch_SMD:SW_MEC_5GSH9
- added D6: LED_GREEN, LED_SMD:LED_0603_1608Metric, F.Cu at (192.8, 93.2)
- added R22: 1k, Resistor_SMD:R_0603_1608Metric, F.Cu at (151.6, 81.0)
- D5: value D_Schottky -> 1N5821
- moved R6 21.9 mm to (191.2, 96.0)
- moved C9 5.92 mm to (150.8, 78.6), turned to 0 degrees
- moved C8 5.90 mm to (153.8, 78.6), turned to 180 degrees
- moved Y1 3.89 mm to (152.6, 75.0)
- moved R8 1.12 mm to (151.5, 101.0)
- moved R9 1.12 mm to (150.0, 101.0)
- moved C37 0.05 mm to (154.0, 101.1)
Connections:
- C9 pad 2: /XOUT -> /crystal r
- R5 pad 2: /sw_r -> Net-(R5-Pad2)
- R6 pad 1: /sw_r -> Net-(R6-Pad1)
- R6 pad 2: /sw_led -> Net-(R6-Pad2)
- Y1 pad 2: /XOUT -> /crystal r
Routing:
- net /sw_r: track 9.53 -> 0.00 mm
- net /XOUT: track 15.8 -> 6.35 mm
- net /1.1V internal rp2040 reg: track 18.9 -> 27.5 mm, vias 0 -> 2
- net /crystal r: track 0.00 -> 7.71 mm
- net /sw_led: track 4.01 -> 0.00 mm
- net /-: track 6.72 -> 5.21 mm
- net /+: track 6.72 -> 5.21 mm
- net /USB_D_P: track 38.7 -> 39.6 mm
- net /USB_D_N: track 41.1 -> 41.8 mm
- net /3.3v rail: track 103.0 -> 103.7 mm, vias 34 -> 32
Other:
- board text added: "SWDIO"
- board text removed: "SWD"
