File: Engineering 2023 UAV flight controller/Engineering 2023 UAV flight controller.kicad_pcb (KiCad board)
At the start: 4 copper layers, 96.9 x 100 mm, 110 parts, among them J1 Micro_SD_Card, J10 DIO, J2 ESC speed control, J3 USB_C_Receptacle_USB2.0, J4 Conn_Coaxial, J5 external power rail, J6 GPIO, J7 external ground rail, J8 Conn_01x03, M1 Aileron Left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

Commit message: E^2
Parts:
- moved C10 0.50 mm to (64.8, 68.6)
Routing:
- net /QSPI_SS: track 0.00 -> 25.4 mm
- net /QSPI_SD1: track 0.00 -> 17.6 mm
- net /QSPI_SD2: track 0.00 -> 12.2 mm
- net /QSPI_SD3: track 0.00 -> 7.19 mm
- net /QSPI_SCLK: track 0.00 -> 5.88 mm
- net /QSPI_SD0: track 0.00 -> 4.93 mm
- net Net-(R5-Pad2): track 0.00 -> 3.61 mm
- net GND: track 111.5 -> 114.7 mm, vias 61 -> 63
Changed lines of the file:
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@@
   )
   (footprint "Capacitor_SMD:C_0603_1608Metric" (layer "F.Cu")
-    (at 64.8 68.1 -90)
+    (at 64.8 68.6 -90)
     (descr "Capacitor SMD 0603 (1608 Metric), square (rectangular) end terminal, IPC_7351 nominal, (Body size source: IPC-SM-782 page 76, https://www.pcb-3d.com/wordpress/wp-content/uploads/ipc-sm-782a_amendment_1_and_2.pdf), generated with kicad-footprint-generator")
     (tags "capacitor")
@@
   (segment (start 64.15 58.15) (end 63.35 58.95) (width 0.2) (layer "F.Cu") (net 2))
   (segment (start 70.75 37.6) (end 70.75 36.8) (width 0.2) (layer "F.Cu") (net 2))
+  (segment (start 53.5 46.4) (end 53.6 46.5) (width 0.2) (layer "F.Cu") (net 2))
   (segment (start 79.6 101.025) (end 79.6 102.2) (width 0.2) (layer "F.Cu") (net 2))
   (segment (start 48.68 39.1) (end 48.68 37.42) (width 0.2) (layer "F.Cu") (net 2))
@@
   (segment (start 53.6 109.2) (end 51 111.8) (width 0.2) (layer "F.Cu") (net 2))
   (segment (start 55.03 37.33) (end 55 37.3) (width 0.2) (layer "F.Cu") (net 2))
+  (segment (start 79.8 65.7) (end 79.8 67.2) (width 0.2) (layer "F.Cu") (net 2))
   (segment (start 72.225 107.2) (end 70.92 105.895) (width 0.2) (layer "F.Cu") (net 2))
   (segment (start 56.025 65.8) (end 54.7 65.8) (width 1) (layer "F.Cu") (net 2))
@@
   (segment (start 97.15 74.855) (end 97.525 74.48) (width 0.2) (layer "F.Cu") (net 2))
   (segment (start 63.15 60.95) (end 64.1 60) (width 0.2) (layer "F.Cu") (net 2))
+  (segment (start 53.5 44.8) (end 53.5 46.4) (width 0.2) (layer "F.Cu") (net 2))
   (segment (start 60.5 68.875) (end 60.5 70.2) (width 1) (layer "F.Cu") (net 2))
   (segment (start 51.34 83.46) (end 54.14 83.46) (width 1) (layer "F.Cu") (net 2))
@@
   (segment (start 66.425 71.925) (end 66.4 71.9) (width 0.2) (layer "F.Cu") (net 2))
   (segment (start 56.025 64.3) (end 54.7 64.3) (width 1) (layer "F.Cu") (net 2))
-  (segment (start 64.8 68.875) (end 64.8 70.1) (width 1) (layer "F.Cu") (net 2))
+  (segment (start 64.8 69.375) (end 64.8 70.6) (width 1) (layer "F.Cu") (net 2))
   (segment (start 55.375 92.2) (end 55.4 92.225) (width 0.2) (layer "F.Cu") (net 2))
   (segment (start 61.3 52.725) (end 61.3 51.4) (width 1) (layer "F.Cu") (net 2))
@@
   (via (at 93 113.6) (size 1) (drill 0.75) (layers "F.Cu" "B.Cu") (net 2))
   (via (at 55.6 111.6) (size 1) (drill 0.75) (layers "F.Cu" "B.Cu") (net 2))
-  (via (at 64.8 70.1) (size 1) (drill 0.75) (layers "F.Cu" "B.Cu") (net 2))
+  (via (at 64.8 70.6) (size 1) (drill 0.75) (layers "F.Cu" "B.Cu") (net 2))
   (via (at 103 72) (size 1) (drill 0.75) (layers "F.Cu" "B.Cu") (net 2))
   (via (at 46.4 115.6) (size 1) (drill 0.75) (layers "F.Cu" "B.Cu") (net 2))
@@
   (via (at 48.7 25.8) (size 1) (drill 0.75) (layers "F.Cu" "B.Cu") (net 2))
   (via (at 76.2 91.4) (size 1) (drill 0.75) (layers "F.Cu" "B.Cu") (net 2))
+  (via (at 79.8 67.2) (size 1) (drill 0.75) (layers "F.Cu" "B.Cu") (net 2))
   (via (at 67 36.8) (size 1) (drill 0.75) (layers "F.Cu" "B.Cu") (net 2))
   (via (at 60.5 70.2) (size 1) (drill 0.75) (layers "F.Cu" "B.Cu") (net 2))
@@
   (via (at 64.2 60) (size 1) (drill 0.75) (layers "F.Cu" "B.Cu") (net 2))
   (via (at 89 39) (size 1) (drill 0.75) (layers "F.Cu" "B.Cu") (net 2))
+  (via (at 53.6 46.5) (size 1) (drill 0.75) (layers "F.Cu" "B.Cu") (net 2))
   (via (at 93.6 74.2) (size 1) (drill 0.75) (layers "F.Cu" "B.Cu") (net 2))
   (via (at 64.2 62) (size 1) (drill 0.75) (layers "F.Cu" "B.Cu") (net 2))
@@
   (segment (start 33.8 84.4) (end 33.9 84.3) (width 0.75) (layer "F.Cu") (net 4))
   (segment (start 40.8 85.95) (end 37.125 82.275) (width 0.75) (layer "F.Cu") (net 4))
-  (segment (start 63.35 64.4175) (end 63.35 65.52) (width 0.2) (layer "F.Cu") (net 5))
   (segment (start 62.55 55.35) (end 62.3 55.1) (width 0.2) (layer "F.Cu") (net 5))
+  (segment (start 64.8 67) (end 64.2 66.4) (width 0.2) (layer "F.Cu") (net 5))
   (segment (start 62.55 56.55) (end 62.55 55.35) (width 0.2) (layer "F.Cu") (net 5))
-  (segment (start 64.8 66.6) (end 64.8 67.325) (width 0.2) (layer "F.Cu") (net 5))
+  (segment (start 63.8 66.4) (end 63.35 65.95) (width 0.2) (layer "F.Cu") (net 5))
   (segment (start 62.3 55.1) (end 61.6 55.1) (width 0.2) (layer "F.Cu") (net 5))
-  (segment (start 63.8 66.4) (end 64.6 66.4) (width 0.2) (layer "F.Cu") (net 5))
   (segment (start 61.3 54.8) (end 61.3 54.275) (width 0.2) (layer "F.Cu") (net 5))
   (segment (start 62.55 58.95) (end 62.5 59) (width 0.12) (layer "F.Cu") (net 5))
-  (segment (start 63.35 65.52) (end 63.35 65.95) (width 0.2) (layer "F.Cu") (net 5))
+  (segment (start 63.35 65.95) (end 63.35 64.4175) (width 0.2) (layer "F.Cu") (net 5))
   (segment (start 63.3 63) (end 63.3 62.9) (width 0.12) (layer "F.Cu") (net 5))
   (segment (start 61.4 63) (end 61.4 62.9) (width 0.12) (layer "F.Cu") (net 5))
   (segment (start 61.35 64.4175) (end 61.35 65.55) (width 0.2) (layer "F.Cu") (net 5))
+  (segment (start 64.8 67.5) (end 64.8 67.325) (width 0.2) (layer "F.Cu") (net 5))
   (segment (start 61.25 65.65) (end 60.5 66.4) (width 0.2) (layer "F.Cu") (net 5))
-  (segment (start 63.35 65.95) (end 63.8 66.4) (width 0.2) (layer "F.Cu") (net 5))
   (segment (start 61.6 55.1) (end 61.3 54.8) (width 0.2) (layer "F.Cu") (net 5))
+  (segment (start 64.8 67.5) (end 64.8 67.825) (width 0.12) (layer "F.Cu") (net 5))
   (segment (start 60.5 66.4) (end 60.5 67.325) (width 0.2) (layer "F.Cu") (net 5))
   (segment (start 62.55 57.5425) (end 62.55 56.55) (width 0.2) (layer "F.Cu") (net 5))
-  (segment (start 64.6 66.4) (end 64.8 66.6) (width 0.2) (layer "F.Cu") (net 5))
+  (segment (start 64.8 67.5) (end 64.8 67) (width 0.2) (layer "F.Cu") (net 5))
+  (segment (start 64.2 66.4) (end 63.8 66.4) (width 0.2) (layer "F.Cu") (net 5))
   (segment (start 61.35 65.55) (end 61.25 65.65) (width 0.2) (layer "F.Cu") (net 5))
   (via (at 62.55 56.55) (size 0.3) (drill 0.2) (layers "F.Cu" "B.Cu") (net 5))
@@
   (segment (start 55.03 21.87) (end 55.03 24.1) (width 0.12) (layer "F.Cu") (net 52))
   (segment (start 56.155 20.745) (end 55.03 21.87) (width 0.12) (layer "F.Cu") (net 52))
+  (segment (start 77.195 70.905) (end 77.6 70.5) (width 0.12) (layer "F.Cu") (net 59))
+  (segment (start 75.175 72.7) (end 75.175 73.525) (width 0.12) (layer "F.Cu") (net 59))
+  (segment (start 67.8 65) (end 67.2175 64.4175) (width 0.12) (layer "F.Cu") (net 59))
+  (segment (start 67.2175 64.4175) (end 65.75 64.4175) (width 0.12) (layer "F.Cu") (net 59))
+  (segment (start 75.2 72.675) (end 75.175 72.7) (width 0.12) (layer "F.Cu") (net 59))
+  (segment (start 75.2 70.905) (end 75.2 72.675) (width 0.12) (layer "F.Cu") (net 59))
+  (segment (start 76.9 65) (end 67.8 65) (width 0.12) (layer "F.Cu") (net 59))
+  (segment (start 75.2 70.905) (end 77.195 70.905) (width 0.12) (layer "F.Cu") (net 59))
+  (segment (start 77.6 65.7) (end 76.9 65) (width 0.12) (layer "F.Cu") (net 59))
+  (segment (start 75.175 73.525) (end 74.5 74.2) (width 0.12) (layer "F.Cu") (net 59))
+  (segment (start 77.6 70.5) (end 77.6 65.7) (width 0.12) (layer "F.Cu") (net 59))
+  (segment (start 74.5 74.2) (end 72.425 74.2) (width 0.12) (layer "F.Cu") (net 59))
+  (segment (start 76.825 72.7) (end 76.825 73.225) (width 0.12) (layer "F.Cu") (net 60))
+  (segment (start 76.825 73.225) (end 77.1 73.5) (width 0.12) (layer "F.Cu") (net 60))
+  (segment (start 77.1 73.5) (end 79.8 73.5) (width 0.12) (layer "F.Cu") (net 60))
   (segment (start 82.125 28.9) (end 93.8 28.9) (width 0.12) (layer "F.Cu") (net 67))
   (segment (start 96.2 26.5) (end 101 26.5) (width 0.12) (layer "F.Cu") (net 67))
@@
   (segment (start 49.5 21.9) (end 49.5 18.2) (width 0.12) (layer "F.Cu") (net 70))
   (segment (start 49.95 22.35) (end 49.5 21.9) (width 0.12) (layer "F.Cu") (net 70))
+  (segment (start 77 66.1) (end 76.2 65.3) (width 0.12) (layer "F.Cu") (net 71))
+  (segment (start 75.2 69.635) (end 76.465 69.635) (width 0.12) (layer "F.Cu") (net 71))
+  (segment (start 65.35 64.751985) (end 65.35 64.4175) (width 0.12) (layer "F.Cu") (net 71))
+  (segment (start 77 69.1) (end 77 66.1) (width 0.12) (layer "F.Cu") (net 71))
+  (segment (start 76.465 69.635) (end 77 69.1) (width 0.12) (layer "F.Cu") (net 71))
+  (segment (start 65.898015 65.3) (end 65.35 64.751985) (width 0.12) (layer "F.Cu") (net 71))
+  (segment (start 76.2 65.3) (end 65.898015 65.3) (width 0.12) (layer "F.Cu") (net 71))
+  (segment (start 75.165 68.4) (end 75.2 68.365) (width 0.12) (layer "F.Cu") (net 72))
+  (segment (start 70.3 65.8) (end 72.9 68.4) (width 0.12) (layer "F.Cu") (net 72))
+  (segment (start 64.95 64.85) (end 65.9 65.8) (width 0.12) (layer "F.Cu") (net 72))
+  (segment (start 64.95 64.4175) (end 64.95 64.85) (width 0.12) (layer "F.Cu") (net 72))
+  (segment (start 65.9 65.8) (end 70.3 65.8) (width 0.12) (layer "F.Cu") (net 72))
+  (segment (start 72.9 68.4) (end 75.165 68.4) (width 0.12) (layer "F.Cu") (net 72))
+  (segment (start 66.595 67.095) (end 64.55 65.05) (width 0.12) (layer "F.Cu") (net 73))
+  (segment (start 64.55 65.05) (end 64.55 64.4175) (width 0.12) (layer "F.Cu") (net 73))
+  (segment (start 68 67.095) (end 66.595 67.095) (width 0.12) (layer "F.Cu") (net 73))
+  (segment (start 64.15 65.1) (end 64.15 64.4175) (width 0.12) (layer "F.Cu") (net 74))
+  (segment (start 67.415 68.365) (end 64.15 65.1) (width 0.12) (layer "F.Cu") (net 74))
+  (segment (start 68 68.365) (end 67.415 68.365) (width 0.12) (layer "F.Cu") (net 74))
+  (segment (start 63.75 65.182304) (end 63.75 64.4175) (width 0.12) (layer "F.Cu") (net 75))
+  (segment (start 66.2 68.2) (end 66.2 67.632304) (width 0.12) (layer "F.Cu") (net 75))
+  (segment (start 68 69.635) (end 67.635 69.635) (width 0.12) (layer "F.Cu") (net 75))
+  (segment (start 67.635 69.635) (end 66.2 68.2) (width 0.12) (layer "F.Cu") (net 75))
+  (segment (start 66.2 67.632304) (end 63.75 65.182304) (width 0.12) (layer "F.Cu") (net 75))
   (segment (start 54.4 102.65) (end 54.55 102.65) (width 0.2) (layer "F.Cu") (net 116))
   (segment (start 54.625 102.575) (end 58 102.575) (width 1) (layer "F.Cu") (net 116))
