File: wearable PDA/wearable PDA.kicad_sch (KiCad schematic)
At the start: 5 parts

Commit message: stuff
Parts:
- removed U? (x5): OSD32MP157C-512M-BAA, footprints:OSD32MP157C-512M-BAA, symbol OSD32MP157C-512M-BAA:OSD32MP157C-512M-BAA
- added U? (x7): STM32MP157FAB1, STM32MP1FAB1:LFBGA354_16X16_STM, symbol STM32MP157FAB1_fun:STM32MP157FAB1
Connections:
- no-connect marks 10 -> 0
