File: calen wah pedal/calen wah pedal.kicad_sch (KiCad schematic)
At the start: 25 parts, among them J1 in jack, J2 AudioJack2_Ground, SW1 SW_DPDT_x2, U1 TL072

Commit message: calen pedel
Parts:
- removed C1, C5: 100uf, symbol Device:C_Polarized
- removed C2: 1uf, symbol Device:C
- removed C6: 0.01u, symbol Device:C
- removed C7, C8: 220nf, symbol Device:C
- removed D1: D, symbol Device:D
- removed J2: AudioJack2_Ground, symbol Connector:AudioJack2_Ground
- removed RV2, RV4: 100k, symbol Device:R_Potentiometer
- removed RV3: 250, symbol Device:R_Potentiometer
- removed SW1: SW_DPDT_x2, symbol Switch:SW_DPDT_x2
- removed U1: TL072, symbol Amplifier_Operational:TL072
- added C1: 0.01u, Capacitor_THT:CP_Axial_L10.0mm_D4.5mm_P15.00mm_Horizontal, symbol Device:C
- added C2: 4u7, Capacitor_THT:CP_Axial_L10.0mm_D4.5mm_P15.00mm_Horizontal, symbol Device:C_Polarized
- added C5: 0.22u, Capacitor_THT:CP_Axial_L10.0mm_D4.5mm_P15.00mm_Horizontal, symbol Device:C
- added J2: 9v in, Connector_BarrelJack:BarrelJack_Horizontal, symbol Connector:Jack-DC
- added J3: out, Connector_Audio:Jack_3.5mm_Lumberg_1503_07_Horizontal, symbol Connector:AudioJack2_Ground
- added Q1, Q2: 2N3904, Package_TO_SOT_THT:TO-92_Inline, symbol Transistor_BJT:2N3904
- added R10: 10k, Resistor_THT:R_Axial_DIN0207_L6.3mm_D2.5mm_P10.16mm_Horizontal, symbol Device:R
- added R8: 470k, Resistor_THT:R_Axial_DIN0207_L6.3mm_D2.5mm_P10.16mm_Horizontal, symbol Device:R
- added R9: 1k, Resistor_THT:R_Axial_DIN0207_L6.3mm_D2.5mm_P10.16mm_Horizontal, symbol Device:R
- C3: value 0.1uf -> 0.22u; footprint (none) -> Capacitor_THT:CP_Axial_L10.0mm_D4.5mm_P15.00mm_Horizontal
- C4: value 220nf -> 0.01u; footprint (none) -> Capacitor_THT:CP_Axial_L10.0mm_D4.5mm_P15.00mm_Horizontal
- J1: value in jack -> in; footprint (none) -> Connector_Audio:Jack_3.5mm_Lumberg_1503_07_Horizontal
- L1: value 500mH -> 500m; footprint (none) -> Inductor_THT:L_Axial_L24.0mm_D7.1mm_P5.08mm_Vertical_Vishay_IM-10-28
- R1: value 100k -> 68k; footprint (none) -> Resistor_THT:R_Axial_DIN0207_L6.3mm_D2.5mm_P10.16mm_Horizontal
- R2: value 100k -> 1k5; footprint (none) -> Resistor_THT:R_Axial_DIN0207_L6.3mm_D2.5mm_P10.16mm_Horizontal
- R3: value 220k -> 22k; footprint (none) -> Resistor_THT:R_Axial_DIN0207_L6.3mm_D2.5mm_P10.16mm_Horizontal
- R4: value 1k -> 470; footprint (none) -> Resistor_THT:R_Axial_DIN0207_L6.3mm_D2.5mm_P10.16mm_Horizontal
- R5: value 1k -> 470k; footprint (none) -> Resistor_THT:R_Axial_DIN0207_L6.3mm_D2.5mm_P10.16mm_Horizontal
- R6: value 100k -> 33k; footprint (none) -> Resistor_THT:R_Axial_DIN0207_L6.3mm_D2.5mm_P10.16mm_Horizontal
- R7: value 470k -> 82k; footprint (none) -> Resistor_THT:R_Axial_DIN0207_L6.3mm_D2.5mm_P10.16mm_Horizontal
- RV1: value 50k -> 100k; footprint (none) -> Potentiometer_THT:Potentiometer_ACP_CA9-H5_Horizontal
Connections:
- net SWA_OUT2 is gone; now on an unnamed net: C4.1
- net GND: now also R4.1, R7.1, RV1.3, C2.2, J2.1, J3.G, J3.T, R10.1; no longer C3.1
- net at C3.2: now also RV1.1, J3.S; no longer R1.1
- net at R2.2: now also C1.2, Q1.2 (B)
- net at R3.1: now also C3.1, R5.2, Q1.3 (C), R8.2; no longer C4.2
- net 9V: now reaches R3.2
- net 9V: now also J2.2, R9.2; no longer R4.1
- net at R6.1: now also L1.2, R2.1; no longer R5.2
- net at R6.2: now also L1.1, R5.1, R7.2, C2.1
- net SWA_in: no longer names the net of J1.S
- net SWA_in: now also R1.1
- removed net V_ref: L1.2, R1.2, R2.1, R5.1, RV1.2, RV1.3
- new net: Q1.1 (E), R4.2
- new net: C5.1, RV1.2
- new net: C1.1, R1.2
- new net: C4.2, Q2.1 (E), R10.2
- new net: C5.2, Q2.2 (B), R8.1
- new net: Q2.3 (C), R9.1
- no-connect marks 1 -> 0
